File: DatassetteAudioAdapter.kicad_pcb (KiCad board)
At the start: 2 copper layers, 41 x 43.6 mm, 20 parts, among them CN1 AUDIO_IN, CN101 AUDIO_IN_JACK, CN2 TAPE_PORT, SW1 SW_INVERT1, U1 CD4049, U2 LM741

Commit message: CassetteAdapter -> DatassetteAudioAdapter
Parts:
- CN1: footprint CassetteAdapter:SWITCHCRAFT_PJRAN1X1U01X -> DatassetteAudioAdapter:SWITCHCRAFT_PJRAN1X1U01X
- CN101: footprint CassetteAdapter:AudioJack_SJ1-3525N -> DatassetteAudioAdapter:AudioJack_SJ1-3525N
- CN2: footprint CassetteAdapter:C64-Cassette-Port-Female -> DatassetteAudioAdapter:C64-Cassette-Port-Female
- RV1: footprint CassetteAdapter:Pot_Bourns_3306P -> DatassetteAudioAdapter:Pot_Bourns_3306P
- V0: footprint CassetteAdapter:cc_by_nc_sa_small -> DatassetteAudioAdapter:cc_by_nc_sa_small
Changed lines of the file:
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@@
     (add_net GND)
   )
-  (module CassetteAdapter:cc_by_nc_sa_small (layer B.Cu)
+  (module DatassetteAudioAdapter:cc_by_nc_sa_small (layer B.Cu)
     (at 144.769166 94.732 180)
     (fp_text reference V0 (at 0 0) (layer B.SilkS) hide
@@
       (xy 3.514499 0.031726) (xy 3.519761 0.049945) (xy 3.568189 0.21665) (xy 3.624095 0.095625)) (layer B.SilkS) (width 0.01))
   )
-  (module CassetteAdapter:AudioJack_SJ1-3525N (layer F.Cu)
+  (module DatassetteAudioAdapter:AudioJack_SJ1-3525N (layer F.Cu)
     (at 148.343 72.262 90)
     (tags "audio jack 3.5mm trs")
@@
     )
   )
-  (module CassetteAdapter:C64-Cassette-Port-Female (layer F.Cu)
+  (module DatassetteAudioAdapter:C64-Cassette-Port-Female (layer F.Cu)
     (at 131.699 109.22)
     (fp_text reference CN2 (at -7.366 -7.112) (layer F.SilkS)
@@
     )
   )
-  (module CassetteAdapter:SWITCHCRAFT_PJRAN1X1U01X (layer F.Cu)
+  (module DatassetteAudioAdapter:SWITCHCRAFT_PJRAN1X1U01X (layer F.Cu)
     (at 144.593 72.262 180)
     (fp_text reference CN1 (at 7.179 4.19) (layer F.SilkS)
@@
     )
   )
-  (module CassetteAdapter:Pot_Bourns_3306P (layer F.Cu)
+  (module DatassetteAudioAdapter:Pot_Bourns_3306P (layer F.Cu)
     (at 138.323 83.352 90)
     (fp_text reference RV1 (at -4.659 0.742 180) (layer F.SilkS)
