File: DatassetteAudioAdapter.sch (KiCad schematic (older format))
At the start: 20 parts, among them CN1 AUDIO_IN, CN101 AUDIO_IN_JACK, CN2 TAPE_PORT, SW1 SW_INVERT1, U1 CD4049, U2 LM741

Commit message: CassetteAdapter -> DatassetteAudioAdapter
Parts:
- CN1: footprint CassetteAdapter:SWITCHCRAFT_PJRAN1X1U01X -> DatassetteAudioAdapter:SWITCHCRAFT_PJRAN1X1U01X
- CN101: footprint CassetteAdapter:AudioJack_SJ1-3525N -> DatassetteAudioAdapter:AudioJack_SJ1-3525N
- CN2: footprint CassetteAdapter:C64-Cassette-Port-Female -> DatassetteAudioAdapter:C64-Cassette-Port-Female
- RV1: footprint CassetteAdapter:Pot_Bourns_3306P -> DatassetteAudioAdapter:Pot_Bourns_3306P
- V0: footprint CassetteAdapter:cc_by_nc_sa_small -> DatassetteAudioAdapter:cc_by_nc_sa_small
Changed lines of the file:
@@
 F 0 "RV1" H 3205 2341 50  0000 R CNN
 F 1 "10k" H 3205 2250 50  0000 R CNN
-F 2 "CassetteAdapter:Pot_Bourns_3306P" H 3275 2295 50  0001 C CNN
+F 2 "DatassetteAudioAdapter:Pot_Bourns_3306P" H 3275 2295 50  0001 C CNN
 F 3 "~" H 3275 2295 50  0001 C CNN
 	1    3275 2295
@@
 F 0 "CN1" H 2183 2621 50  0000 C CNN
 F 1 "AUDIO_IN" H 2183 2530 50  0000 C CNN
-F 2 "CassetteAdapter:SWITCHCRAFT_PJRAN1X1U01X" H 2175 2240 50  0001 L BNN
+F 2 "DatassetteAudioAdapter:SWITCHCRAFT_PJRAN1X1U01X" H 2175 2240 50  0001 L BNN
 F 3 "A" H 2175 2240 50  0001 L BNN
 F 4 "Switchcraft" H 2175 2240 50  0001 L BNN "Field4"
@@
 F 0 "CN101" H 1151 2073 50  0000 R CNN
 F 1 "AUDIO_IN_JACK" H 1151 2164 50  0000 R CNN
-F 2 "CassetteAdapter:AudioJack_SJ1-3525N" H 1430 2240 50  0001 C CNN
+F 2 "DatassetteAudioAdapter:AudioJack_SJ1-3525N" H 1430 2240 50  0001 C CNN
 F 3 "~" H 1430 2240 50  0001 C CNN
 	1    1430 2240
@@
 F 0 "V0" H 10668 6426 50  0000 L CNN
 F 1 "OSHW_LOGO" H 10668 6335 50  0000 L CNN
-F 2 "CassetteAdapter:cc_by_nc_sa_small" H 10590 6380 50  0001 C CNN
+F 2 "DatassetteAudioAdapter:cc_by_nc_sa_small" H 10590 6380 50  0001 C CNN
 F 3 "" H 10590 6380 50  0001 C CNN
 F 4 "---" H 10590 6380 50  0001 C CNN "MouserPN"
@@
 F 0 "CN2" H 10642 2369 50  0000 R CNN
 F 1 "TAPE_PORT" H 10642 2278 50  0000 R CNN
-F 2 "CassetteAdapter:C64-Cassette-Port-Female" H 10670 2395 50  0001 C CNN
+F 2 "DatassetteAudioAdapter:C64-Cassette-Port-Female" H 10670 2395 50  0001 C CNN
 F 3 "~" H 10670 2395 50  0001 C CNN
 	1    10670 2395
